File: EcoIDSwitch/EcoIDSwitch.kicad_pcb (KiCad board)
At the start: 2 copper layers, 12.7 x 33.7 mm, 2 parts, among them J1 Conn_02x08_Counter_Clockwise, SW1 SW_DIP_x08

Commit message: Refactor solder PCB to same dimensions as switch PCB
Other:
- board text added: "BBC EcoID Switch v0.2"
- board text removed: "BBC EcoID Switch v0.1"
Changed lines of the file:
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@@
   (gr_line (start 168.1 101.8) (end 168.1 68.1) (layer "Edge.Cuts") (width 0.1))
   (gr_line (start 155.4 101.8) (end 168.1 101.8) (layer "Edge.Cuts") (width 0.1))
-  (gr_text "BBC EcoID\nSwitch\nv0.1" (at 161.75 95.68) (layer "B.SilkS")
+  (gr_text "BBC EcoID\nSwitch\nv0.2" (at 161.75 95.68) (layer "B.SilkS")
     (effects (font (size 1.5 1.5) (thickness 0.3)) (justify mirror))
   )
